Commit message: cobot ros package

File: mycobot_ros/mycobot_description/urdf/mycobot_320_m5_2022/new_mycobot_pro_320moveit_m5_2022.urdf (robot description, URDF)
Before this commit: robot firefighter, 7 links, 6 joints
Links:
- added link ardconv_link; collision box size=0.38 0.18 0.1; visual mesh filename=package://mycobot_description/urdf/mycobot_320_m5_2022/ardc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
- added link base_link; collision box size=1.5 1.5 0.0000000001; visual box size=1.5 1.5 0.0000000001
- added link big_box_link1; visual mesh filename=package://mycobot_description/urdf/mycobot_320_m5_2022/big_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
- added link big_box_link2; visual mesh filename=package://mycobot_description/urdf/mycobot_320_m5_2022/big_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
- added link box_link; collision box size=0.2 0.2 0.06; visual mesh filename=package://mycobot_description/urdf/mycobot_320_m5_2022/box_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
- added link box_link2; collision box size=0.2 0.2 0.06; visual mesh filename=package://mycobot_description/urdf/mycobot_320_m5_2022/box_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
- added link camera_link; collision box size=0.05 0.13 0.02; visual mesh filename=package://mycobot_description/urdf/mycobot_320_m5_2022/grip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
- added link conv_link; collision box size=0.65 0.15 0.2; visual mesh filename=package://mycobot_description/urdf/mycobot_320_m5_2022/conv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
- added link conv_link2; collision box size=0.65 0.15 0.2; visual mesh filename=package://mycobot_description/urdf/mycobot_320_m5_2022/conv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
- added link desk_link; collision box size=0.6 0.35 0.1; visual mesh filename=package://mycobot_description/urdf/mycobot_320_m5_2022/desk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
- added link gripper_base; collision cylinder length=0.13 radius=0.0195; visual mesh filename=package://mycobot_description/urdf/mycobot_320_m5_2022/grip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
- added link gripper_left1; collision cylinder length=0.02 radius=0.047; visual mesh filename=package://mycobot_description/urdf/mycobot_320_m5_2022/grip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
- added link gripper_left2; collision cylinder length=0.08 radius=0.025; visual mesh filename=package://mycobot_description/urdf/mycobot_320_m5_2022/grip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
- added link gripper_left3; collision cylinder length=0.02 radius=0.01; visual mesh filename=package://mycobot_description/urdf/mycobot_320_m5_2022/grip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
- added link gripper_right1; collision cylinder length=0.02 radius=0.047; visual mesh filename=package://mycobot_description/urdf/mycobot_320_m5_2022/grip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
- added link gripper_right2; collision cylinder length=0.08 radius=0.025; visual mesh filename=package://mycobot_description/urdf/mycobot_320_m5_2022/grip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
- added link gripper_right3; collision cylinder length=0.02 radius=0.01; visual mesh filename=package://mycobot_description/urdf/mycobot_320_m5_2022/grip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
- added link reader_link; collision box size=0.1 0.14 0.1; visual mesh filename=package://mycobot_description/urdf/mycobot_320_m5_2022/read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
- link base: geometry collision cylinder length=0.096 radius=0.07; visual mesh filename=package://mycobot_description/urdf/mycobot_320_m5_2022/base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
- link link1: geometry collision cylinder length=0.114 radius=0.0382; visual mesh filename=package://mycobot_description/urdf/mycobot_320_m5_2022/link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
- link link2: geometry collision cylinder length=0.203 radius=0.0382; visual mesh filename=package://mycobot_description/urdf/mycobot_320_m5_2022/link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
- link link3: geometry collision cylinder length=0.18 radius=0.032; visual mesh filename=package://mycobot_description/urdf/mycobot_320_m5_2022/link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
- link link4: geometry collision cylinder length=0.073 radius=0.029; visual mesh filename=package://mycobot_description/urdf/mycobot_320_m5_2022/link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
- link link5: geometry collision cylinder length=0.078 radius=0.046; visual mesh filename=package://mycobot_description/urdf/mycobot_320_m5_2022/link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
Joints:
- added joint desk_base: type fixed, parent base, child desk_link, origin xyz=-0.35 -0.175 -0.05 rpy=0 0 0, axis 0 0 0
- added joint gripper_base_to_gripper_left2: type fixed, parent gripper_base, child gripper_left2, origin xyz=-0.05 -0.01 0 rpy=0 0 0, axis 0 0 1, limit lower=-0.8 upper=0.5 effort=1000.0 velocity=0, mimic joint=gripper_controller multiplier=1.0 offset=0
- added joint gripper_base_to_gripper_right2: type fixed, parent gripper_base, child gripper_right2, origin xyz=0.046 -0.01 0 rpy=0 0 0, axis 0 0 1, limit lower=-0.5 upper=0.8 effort=1000.0 velocity=0, mimic joint=gripper_controller multiplier=-1.0 offset=0
- added joint gripper_base_to_gripper_right3: type fixed, parent gripper_base, child gripper_right3, origin xyz=0.018 0.016 0 rpy=0 0 0, axis 0 0 1, limit lower=-0.3 upper=0.7 effort=1000.0 velocity=0, mimic joint=gripper_controller multiplier=-1.0 offset=0
- added joint gripper_controller: type fixed, parent gripper_base, child gripper_left3, origin xyz=-0.018 0.016 0 rpy=0 0 0, axis 0 0 1, limit lower=-0.7 upper=0.3 effort=1000.0 velocity=0
- added joint gripper_left3_to_gripper_left1: type fixed, parent gripper_left3, child gripper_left1, origin xyz=-0.0356 0.051 -0.018 rpy=0 0 0, axis 0 0 1, limit lower=-0.5 upper=0.5 effort=1000.0 velocity=0, mimic joint=gripper_controller multiplier=-1.0 offset=0
- added joint gripper_right3_to_gripper_right1: type fixed, parent gripper_right3, child gripper_right1, origin xyz=0.033 0.051 -0.018 rpy=0 0 0, axis 0 0 1, limit lower=-0.5 upper=0.5 effort=1000.0 velocity=0, mimic joint=gripper_controller multiplier=1.0 offset=0
- added joint joint_ardconv: type fixed, parent base_link, child ardconv_link, origin xyz=-0.31 -0.1 0 rpy=0 0 0, axis 0 0 0
- added joint joint_base: type fixed, parent desk_link, child base_link, origin xyz=0.3 0.17 -0.13 rpy=0 0 0, axis 0 0 0
- added joint joint_bigbox1: type fixed, parent base_link, child big_box_link1, origin xyz=0.33 0.2 0 rpy=0 0 0, axis 0 0 0
- added joint joint_bigbox2: type fixed, parent base_link, child big_box_link2, origin xyz=0.01 0.2 0 rpy=0 0 0, axis 0 0 0
- added joint joint_box: type fixed, parent conv_link, child box_link, origin xyz=-0.07 0.65 0.21 rpy=0 0 0, axis 0 0 0
- added joint joint_box2: type fixed, parent conv_link2, child box_link2, origin xyz=-0.07 0.65 0.21 rpy=0 0 0, axis 0 0 0
- added joint joint_camera_to_gripper_base: type fixed, parent camera_link, child gripper_base, origin xyz=0 -0.0385 -0.007 rpy=3.1416 0 0
- added joint joint_camera_to_link6: type fixed, parent link6, child camera_link, origin xyz=0 0 0.015 rpy=-1.5708 0 3.14159
- added joint joint_conv: type fixed, parent base_link, child conv_link, origin xyz=0.09 -0.828 0 rpy=0 0 0, axis 0 0 0
- added joint joint_conv2: type fixed, parent base_link, child conv_link2, origin xyz=-0.17 -0.828 0 rpy=0 0 0, axis 0 0 0
- added joint joint_reader: type fixed, parent base_link, child reader_link, origin xyz=-0.41 0.08 0 rpy=0 0 0, axis 0 0 0
